File: opamp-lc-meter.sch (KiCad schematic (older format))
At the start: 18 parts, among them J1 Conn_01x04, J2 Conn_02x04_Counter_Clockwise, J3 Conn_02x04_Counter_Clockwise, J4 Conn_01x02, J5 Conn_01x02, U1 LM393

Commit message: Change footprint of component socket to an actual socket
Parts:
- J2, J3: footprint Package_DIP:DIP-8_W7.62mm_LongPads -> Package_DIP:DIP-8_W7.62mm_Socket_LongPads
Changed lines of the file:
@@
 F 0 "J2" H 3200 4117 50  0000 C CNN
 F 1 "Conn_02x04_Counter_Clockwise" H 3200 4026 50  0000 C CNN
-F 2 "Package_DIP:DIP-8_W7.62mm_LongPads" H 3150 3800 50  0001 C CNN
+F 2 "Package_DIP:DIP-8_W7.62mm_Socket_LongPads" H 3150 3800 50  0001 C CNN
 F 3 "~" H 3150 3800 50  0001 C CNN
 	1    3150 3800
@@
 F 0 "J3" H 3200 4817 50  0000 C CNN
 F 1 "Conn_02x04_Counter_Clockwise" H 3200 4726 50  0000 C CNN
-F 2 "Package_DIP:DIP-8_W7.62mm_LongPads" H 3150 4500 50  0001 C CNN
+F 2 "Package_DIP:DIP-8_W7.62mm_Socket_LongPads" H 3150 4500 50  0001 C CNN
 F 3 "~" H 3150 4500 50  0001 C CNN
 	1    3150 4500
